Commit message: Added controller for AGV to drive robot via cmd/vel

File: ros2_rm_robot/dual_rm_gazebo/config/dual_rm_75b_gazebo.urdf.xacro (robot description, xacro)
@@ -1,152 +1,175 @@
 <?xml version="1.0"?>
 <robot xmlns:xacro="http://www.ros.org/wiki/xacro" name="dual_rm_75b_gazebo">
-    <link name="world"/>
-    <joint name="fixed" type="fixed">
-        <parent link="world"/>
-        <child link="base_link_underpan"/>
-    </joint>
     <xacro:include filename="$(find dual_rm_75b_description)/urdf/dual_rm_75b_description.urdf.xacro" />
     <gazebo reference="base_link">
         <self_collide>false</self_collide>
-        <gravity>false</gravity>
+        <gravity>true</gravity>
     </gazebo>
     <gazebo reference="r_link1">
         <self_collide>false</self_collide>
-        <gravity>false</gravity>
+        <gravity>true</gravity>
     </gazebo>
     <gazebo reference="r_link2">
         <self_collide>false</self_collide>
-        <gravity>false</gravity>
+        <gravity>true</gravity>
     </gazebo>
     <gazebo reference="r_link3">
         <self_collide>false</self_collide>
-        <gravity>false</gravity>
+        <gravity>true</gravity>
     </gazebo>
     <gazebo reference="r_link4">
         <self_collide>false</self_collide>
-        <gravity>false</gravity>
+        <gravity>true</gravity>
     </gazebo>
     <gazebo reference="r_link5">
         <self_collide>false</self_collide>
-        <gravity>false</gravity>
+        <gravity>true</gravity>
     </gazebo>
     <gazebo reference="r_link6">
         <self_collide>false</self_collide>
-        <gravity>false</gravity>
+        <gravity>true</gravity>
     </gazebo>
     <gazebo reference="r_link7">
         <self_collide>false</self_collide>
-        <gravity>false</gravity>
+        <gravity>true</gravity>
     </gazebo>
     <gazebo reference="l_link1">
         <self_collide>false</self_collide>
-        <gravity>false</gravity>
+        <gravity>true</gravity>
     </gazebo>
     <gazebo reference="l_link2">
         <self_collide>false</self_collide>
-        <gravity>false</gravity>
+        <gravity>true</gravity>
     </gazebo>
     <gazebo reference="l_link3">
         <self_collide>false</self_collide>
-        <gravity>false</gravity>
+        <gravity>true</gravity>
     </gazebo>
     <gazebo reference="l_link4">
         <self_collide>false</self_collide>
-        <gravity>false</gravity>
+        <gravity>true</gravity>
     </gazebo>
     <gazebo reference="l_link5">
         <self_collide>false</self_collide>
-        <gravity>false</gravity>
+        <gravity>true</gravity>
     </gazebo>
     <gazebo reference="l_link6">
         <self_collide>false</self_collide>
-        <gravity>false</gravity>
+        <gravity>true</gravity>
     </gazebo>
     <gazebo reference="l_link7">
         <self_collide>false</self_collide>
-        <gravity>false</gravity>
+        <gravity>true</gravity>
     </gazebo>
     <gazebo reference="head_link1">
         <self_collide>false</self_collide>
-        <gravity>false</gravity>
+        <gravity>true</gravity>
     </gazebo>
     <gazebo reference="head_link2">
         <self_collide>false</self_collide>
-        <gravity>false</gravity>
+        <gravity>true</gravity>
     </gazebo>
     <gazebo reference="camera_link">
         <self_collide>false</self_collide>
-        <gravity>false</gravity>
+        <gravity>true</gravity>
     </gazebo>
     <gazebo reference="link_right_wheel">
         <self_collide>false</self_collide>
-        <gravity>false</gravity>
+        <gravity>true</gravity>
+        <mu1>10.0</mu1>
+        <mu2>10.0</mu2>
+        <kp>1000000.0</kp>
+        <kd>1.0</kd>
+        <minDepth>0.001</minDepth>
+        <maxVel>1.0</maxVel>
     </gazebo>
     <gazebo reference="link_left_wheel">
         <self_collide>false</self_collide>
-        <gravity>false</gravity>
+        <gravity>true</gravity>
+        <mu1>10.0</mu1>
+        <mu2>10.0</mu2>
+        <kp>1000000.0</kp>
+        <kd>1.0</kd>
+        <minDepth>0.001</minDepth>
+        <maxVel>1.0</maxVel>
     </gazebo>
     <gazebo reference="link_swivel_wheel_1_1">
         <self_collide>false</self_collide>
-        <gravity>false</gravity>
+        <gravity>true</gravity>
+        <mu1>0.0</mu1>
+        <mu2>0.0</mu2>
     </gazebo>
     <gazebo reference="link_swivel_wheel_1_2">
         <self_collide>false</self_collide>
-        <gravity>false</gravity>
+        <gravity>true</gravity>
+        <mu1>0.0</mu1>
+        <mu2>0.0</mu2>
     </gazebo>
     <gazebo reference="link_swivel_wheel_2_1">
         <self_collide>false</self_collide>
-        <gravity>false</gravity>
+        <gravity>true</gravity>
+        <mu1>0.0</mu1>
+        <mu2>0.0</mu2>
     </gazebo>
     <gazebo reference="link_swivel_wheel_2_2">
         <self_collide>false</self_collide>
-        <gravity>false</gravity>
+        <gravity>true</gravity>
+        <mu1>0.0</mu1>
+        <mu2>0.0</mu2>
     </gazebo>
     <gazebo reference="link_swivel_wheel_3_1">
         <self_collide>false</self_collide>
-        <gravity>false</gravity>
+        <gravity>true</gravity>
+        <mu1>0.0</mu1>
+        <mu2>0.0</mu2>
     </gazebo>
     <gazebo reference="link_swivel_wheel_3_2">
         <self_collide>false</self_collide>
-        <gravity>false</gravity>
+        <gravity>true</gravity>
+        <mu1>0.0</mu1>
+        <mu2>0.0</mu2>
     </gazebo>
     <gazebo reference="link_swivel_wheel_4_1">
         <self_collide>false</self_collide>
-        <gravity>false</gravity>
+        <gravity>true</gravity>
+        <mu1>0.0</mu1>
+        <mu2>0.0</mu2>
     </gazebo>
     <gazebo reference="link_swivel_wheel_4_2">
         <self_collide>false</self_collide>
-        <gravity>false</gravity>
+        <gravity>true</gravity>
+        <mu1>0.0</mu1>
+        <mu2>0.0</mu2>
     </gazebo>
     <gazebo reference="body_base_link">
         <self_collide>false</self_collide>
-        <gravity>false</gravity>
+        <gravity>true</gravity>
     </gazebo>
     <gazebo reference="platform_base_link">
         <self_collide>false</self_collide>
-        <gravity>false</gravity>
+        <gravity>true</gravity>
     </gazebo>
     <gazebo reference="l_base_link1">
         <self_collide>false</self_collide>
-        <gravity>false</gravity>
+        <gravity>true</gravity>
     </gazebo>
     <gazebo reference="r_base_link1">
         <self_collide>false</self_collide>
-        <gravity>false</gravity>
+        <gravity>true</gravity>
     </gazebo>
     <gazebo reference="r_hand_base_link">
         <self_collide>false</self_collide>
-        <gravity>false</gravity>
+        <gravity>true</gravity>
     </gazebo>
     <gazebo reference="l_hand_base_link">
         <self_collide>false</self_collide>
-        <gravity>false</gravity>
+        <gravity>true</gravity>
     </gazebo>
     <gazebo reference="base_link_underpan">
         <self_collide>false</self_collide>
-        <gravity>false</gravity>
+        <gravity>true</gravity>
     </gazebo>
     <gazebo>
-        <is_static>true</is_static>
+        <is_static>false</is_static>
         <self_collide>true</self_collide>
     </gazebo>
@@ -275,5 +298,5 @@
         </joint>
         <joint name="joint_right_wheel">
-            <command_interface name="position"/>
+            <command_interface name="velocity"/>
             <state_interface name="position">
                 <param name="initial_value">0</param>
@@ -282,11 +305,11 @@
         </joint>
         <joint name="joint_left_wheel">
-            <command_interface name="position"/>
-            <state_interface name="position">
-                <param name="initial_value">0</param>
-            </state_interface>
-            <state_interface name="velocity"/>
-        </joint>
-        <joint name="joint_swivel_wheel_1_1">
+            <command_interface name="velocity"/>
+            <state_interface name="position">
+                <param name="initial_value">0</param>
+            </state_interface>
+            <state_interface name="velocity"/>
+        </joint>
+        <!-- <joint name="joint_swivel_wheel_1_1">
             <command_interface name="position"/>
             <state_interface name="position">
@@ -343,5 +366,5 @@
             </state_interface>
             <state_interface name="velocity"/>
-        </joint>
+        </joint>  -->
     </ros2_control>
     <gazebo>

Commit message: Fixed MOveIt clocked sync and swivel wheel controller for MoveIt

File: ros2_rm_robot/dual_rm_gazebo/config/dual_rm_75b_gazebo.urdf.xacro (robot description, xacro)
@@ -311,6 +311,6 @@
             <state_interface name="velocity"/>
         </joint>
-        <!-- <joint name="joint_swivel_wheel_1_1">
-            <command_interface name="position"/>
+        <joint name="joint_swivel_wheel_1_1">
+            <command_interface name="velocity"/>
             <state_interface name="position">
                 <param name="initial_value">0</param>
@@ -319,5 +319,5 @@
         </joint>
         <joint name="joint_swivel_wheel_1_2">
-            <command_interface name="position"/>
+            <command_interface name="velocity"/>
             <state_interface name="position">
                 <param name="initial_value">0</param>
@@ -326,5 +326,5 @@
         </joint>
         <joint name="joint_swivel_wheel_2_1">
-            <command_interface name="position"/>
+            <command_interface name="velocity"/>
             <state_interface name="position">
                 <param name="initial_value">0</param>
@@ -333,5 +333,5 @@
         </joint>
         <joint name="joint_swivel_wheel_2_2">
-            <command_interface name="position"/>
+            <command_interface name="velocity"/>
             <state_interface name="position">
                 <param name="initial_value">0</param>
@@ -340,5 +340,5 @@
         </joint>
         <joint name="joint_swivel_wheel_3_1">
-            <command_interface name="position"/>
+            <command_interface name="velocity"/>
             <state_interface name="position">
                 <param name="initial_value">0</param>
@@ -347,5 +347,5 @@
         </joint>
         <joint name="joint_swivel_wheel_3_2">
-            <command_interface name="position"/>
+            <command_interface name="velocity"/>
             <state_interface name="position">
                 <param name="initial_value">0</param>
@@ -354,5 +354,5 @@
         </joint>
         <joint name="joint_swivel_wheel_4_1">
-            <command_interface name="position"/>
+            <command_interface name="velocity"/>
             <state_interface name="position">
                 <param name="initial_value">0</param>
@@ -361,10 +361,10 @@
         </joint>
         <joint name="joint_swivel_wheel_4_2">
-            <command_interface name="position"/>
-            <state_interface name="position">
-                <param name="initial_value">0</param>
-            </state_interface>
-            <state_interface name="velocity"/>
-        </joint>  -->
+            <command_interface name="velocity"/>
+            <state_interface name="position">
+                <param name="initial_value">0</param>
+            </state_interface>
+            <state_interface name="velocity"/>
+        </joint>
     </ros2_control>
     <gazebo>
