Commit message: Removed the fixed hands

File: ros2_rm_robot/dual_rm_description/dual_rm_75b_description/urdf/dual_rm_75b_description.urdf.xacro (robot description, xacro)
@@ -4,6 +4,6 @@
   <xacro:include filename="$(find dual_rm_75b_description)/urdf/woosh_agv.urdf.xacro"/>
   <xacro:include filename="$(find dual_rm_75b_description)/urdf/body_head_platform.urdf.xacro"/>
-  <xacro:include filename="$(find dual_rm_75b_description)/urdf/left_hand.urdf.xacro"/>
-  <xacro:include filename="$(find dual_rm_75b_description)/urdf/right_hand.urdf.xacro"/>
+  <!-- <xacro:include filename="$(find dual_rm_75b_description)/urdf/left_hand.urdf.xacro"/> -->
+  <!-- <xacro:include filename="$(find dual_rm_75b_description)/urdf/right_hand.urdf.xacro"/> -->
   <xacro:include filename="$(find dual_rm_75b_description)/urdf/rm75_b_v_left.urdf.xacro"/>
   <xacro:include filename="$(find dual_rm_75b_description)/urdf/rm75_b_v_right.urdf.xacro"/>

File: ros2_rm_robot/dual_rm_gazebo/config/dual_rm_75b_gazebo.urdf.xacro (robot description, xacro)
@@ -2,4 +2,5 @@
 <robot xmlns:xacro="http://www.ros.org/wiki/xacro" name="dual_rm_75b_gazebo">
     <xacro:include filename="$(find dual_rm_75b_description)/urdf/dual_rm_75b_description.urdf.xacro" />
+    <!-- <xacro:include filename="$(find dual_rm_gazebo)/config/dg4f_gazebo_classic.urdf.xacro"/> -->
     <gazebo reference="base_link">
         <self_collide>false</self_collide>
@@ -30,8 +31,8 @@
         <gravity>true</gravity>
     </gazebo>
-    <gazebo reference="r_link7">
-        <self_collide>false</self_collide>
-        <gravity>true</gravity>
-    </gazebo>
+    <!-- <gazebo reference="r_link7">
+        <self_collide>false</self_collide>
+        <gravity>true</gravity>
+    </gazebo> -->
     <gazebo reference="l_link1">
         <self_collide>false</self_collide>
@@ -58,8 +59,8 @@
         <gravity>true</gravity>
     </gazebo>
-    <gazebo reference="l_link7">
-        <self_collide>false</self_collide>
-        <gravity>true</gravity>
-    </gazebo>
+    <!-- <gazebo reference="l_link7">
+        <self_collide>false</self_collide>
+        <gravity>true</gravity>
+    </gazebo> -->
     <gazebo reference="head_link1">
         <self_collide>false</self_collide>
@@ -170,4 +171,9 @@
         <gravity>true</gravity>
     </gazebo>
+    <!-- <xacro:dg4f_attach
+        parent="l_hand_link"
+        xyz="0 0 0.01"
+        rpy="0 0 0"/>
+     -->
     <gazebo>
         <is_static>false</is_static>

File: ros2_rm_robot/dual_rm_moveit_config/dual_rm_75b_moveit_config/config/dual_rm_75b_description.ros2_control.xacro (robot description, xacro)
@@ -50,5 +50,5 @@
                 <state_interface name="velocity"/>
             </joint>
-            <joint name="l_joint7">
+            <!-- <joint name="l_joint7">
                 <command_interface name="position"/>
                 <state_interface name="position">
@@ -56,5 +56,5 @@
                 </state_interface>
                 <state_interface name="velocity"/>
-            </joint>
+            </joint> -->
             <joint name="r_joint1">
                 <command_interface name="position"/>
@@ -99,5 +99,5 @@
                 <state_interface name="velocity"/>
             </joint>
-            <joint name="r_joint7">
+            <!-- <joint name="r_joint7">
                 <command_interface name="position"/>
                 <state_interface name="position">
@@ -105,5 +105,5 @@
                 </state_interface>
                 <state_interface name="velocity"/>
-            </joint>
+            </joint> -->
             <joint name="platform_joint">
                 <command_interface name="position"/>
